File: CircuitDesign/DougsDino/DougsDino.sch (KiCad schematic (older format))
At the start: 101 parts, among them IC1 TPS5420QDRQ1, IC2 TPS5420QDRQ1, IC3 LP2989IMX-5.0_NOPB, IC4 LP2989IMX-3.3_NOPB, IC5 ZXMS6004DN8-13, IC6 ZXMS6004DN8-13, IC7 PCM1725U, IC8 OPA2141AID, IC9 PGA2311U, J1 TB004-750-02GR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

Commit message: Sheet Adjustment
Enlarged the Schematic Sheet in order to fit all of the components.
Other:
- note added: "Audio"
- note added: "Digital"
- note added: "POWER"
- note added: "Relays"
- moved on the sheet: C1, C10, C11, C12, C13, C14, C15, C16, C17, C18, C19, C2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
